File: GRBL Shield.sch (EAGLE design)
At the start: 38 parts

Commit message: Added values for components and added 5V regulator #1
Parts:
- added C4: 100uf, rcl:CPOL-EUE2.5-7
- added IC1: 7805, linear:786TV
- C1, C2, C3: value (none) -> 100uf
- LED1, LED4: value (none) -> RED
- LED2, LED5: value (none) -> GRN
- LED3, LED6: value (none) -> YLW
- LED7: value (none) -> BLU
- R1, R2, R3, R4, R5, R6: value (none) -> 150R
- R10, R8, R9: value (none) -> 10k
- R7: value (none) -> 68R
- SV10: value (none) -> 8-13/GND/AREF
- SV11: value (none) -> A0-A5
- SV12: value (none) -> RST/3.3/5/GND/GND/VIN
- SV9: value (none) -> 0-7
Connections:
- net +24V: now also IC1.VI
- net +5V: now also C4.+, IC1.VO
- net GND: now also C4.-, IC1.GND
Other:
- moved on the sheet: JP1, LED1, LED2, LED3, LED4, LED6, LED7, R1, R10, R2, R3, R4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
